File: Hardware/Electronics/tinyGlow.kicad_pcb (KiCad board)
At the start: 2 copper layers, 48.3 x 48.3 mm, 56 parts, among them IC1 RT6255BHGJ6F, IC2 RT6255BHGJ6F, IC3 RT6255BHGJ6F, IC4 LS0504EVT233, IC5 LS0504EVT233, IC6 LS0504EVT233, J1 Screw_Terminal_01x02, J2 Conn_01x08, J3 Conn_01x09, J4 Conn_01x08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

Commit message: Updated tinyGlow Schematics
Parts:
- removed G***: LOGO, logos.preety:openSource
